File: boat_lights_breakout/reciever_board.sch (EAGLE design)
At the start: 12 parts, among them U1 LM2574HVM-3.3/NOPBNPA0014B_M, U2 LTC5508ESC6TRMPBFSOT-6_SC_LIT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, U3 SN74AUC1G80DCKRDCK5-M, U4 STCS1PHRPOWERSO-8_STM-M, U5 CDBW46-GCDBW-M

Commit message: made progress on reciever board
Parts:
- added C4, C5, C6: (no value), rcl:C-USC0603
Connections:
- net N$1 renamed TOGGLE
- new net N$2: C4.2, U2.RFIN
- net +3V3: now also C5.1, C6.1
- net GND: now also C5.2, C6.2
Changed lines of the file:
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@@
 <part name="GND6" library="supply1" library_urn="urn:adsk.eagle:library:371" deviceset="GND" device=""/>
 <part name="C3" library="rcl" library_urn="urn:adsk.eagle:library:334" deviceset="C-US" device="C0603" package3d_urn="urn:adsk.eagle:package:23616/2"/>
+<part name="+3V3" library="supply1" library_urn="urn:adsk.eagle:library:371" deviceset="+3V3" device=""/>
+<part name="C4" library="rcl" library_urn="urn:adsk.eagle:library:334" deviceset="C-US" device="C0603" package3d_urn="urn:adsk.eagle:package:23616/2"/>
+<part name="C5" library="rcl" library_urn="urn:adsk.eagle:library:334" deviceset="C-US" device="C0603" package3d_urn="urn:adsk.eagle:package:23616/2"/>
+<part name="C6" library="rcl" library_urn="urn:adsk.eagle:library:334" deviceset="C-US" device="C0603" package3d_urn="urn:adsk.eagle:package:23616/2"/>
 </parts>
 <sheets>
@@
 <attribute name="VALUE" x="83.5406" y="174.2186" size="2.0828" layer="96" ratio="6" rot="SR0"/>
 </instance>
-<instance part="+3V1" gate="G$1" x="175.26" y="50.8" smashed="yes">
-<attribute name="VALUE" x="172.72" y="45.72" size="1.778" layer="96" rot="R90"/>
+<instance part="+3V1" gate="G$1" x="160.02" y="27.94" smashed="yes">
+<attribute name="VALUE" x="162.56" y="22.86" size="1.778" layer="96" rot="R90"/>
 </instance>
 <instance part="P+1" gate="1" x="38.1" y="210.82" smashed="yes">
@@
 <attribute name="NAME" x="67.056" y="158.115" size="1.778" layer="95"/>
 <attribute name="VALUE" x="67.056" y="153.289" size="1.778" layer="96"/>
+</instance>
+<instance part="+3V3" gate="G$1" x="88.9" y="45.72" smashed="yes">
+<attribute name="VALUE" x="86.36" y="40.64" size="1.778" layer="96" rot="R90"/>
+</instance>
+<instance part="C4" gate="G$1" x="160.02" y="35.56" smashed="yes" rot="R270">
+<attribute name="NAME" x="160.655" y="34.544" size="1.778" layer="95" rot="R270"/>
+<attribute name="VALUE" x="155.829" y="34.544" size="1.778" layer="96" rot="R270"/>
+</instance>
+<instance part="C5" gate="G$1" x="88.9" y="35.56" smashed="yes">
+<attribute name="NAME" x="89.916" y="36.195" size="1.778" layer="95"/>
+<attribute name="VALUE" x="89.916" y="31.369" size="1.778" layer="96"/>
+</instance>
+<instance part="C6" gate="G$1" x="93.98" y="35.56" smashed="yes">
+<attribute name="NAME" x="94.996" y="36.195" size="1.778" layer="95"/>
+<attribute name="VALUE" x="94.996" y="31.369" size="1.778" layer="96"/>
 </instance>
 </instances>
@@
 <pinref part="U2" gate="A" pin="GND_2"/>
 <pinref part="GND3" gate="1" pin="GND"/>
-<wire x1="99.06" y1="30.48" x2="86.36" y2="30.48" width="0.1524" layer="91"/>
+<wire x1="99.06" y1="30.48" x2="93.98" y2="30.48" width="0.1524" layer="91"/>
+<pinref part="C5" gate="G$1" pin="2"/>
+<wire x1="93.98" y1="30.48" x2="88.9" y2="30.48" width="0.1524" layer="91"/>
+<wire x1="88.9" y1="30.48" x2="86.36" y2="30.48" width="0.1524" layer="91"/>
+<junction x="88.9" y="30.48"/>
+<pinref part="C6" gate="G$1" pin="2"/>
+<junction x="93.98" y="30.48"/>
 </segment>
 <segment>
@@
 <net name="+3V3" class="0">
 <segment>
-<pinref part="U2" gate="A" pin="VCC"/>
-<wire x1="154.94" y1="27.94" x2="154.94" y2="20.32" width="0.1524" layer="91"/>
-<wire x1="154.94" y1="20.32" x2="175.26" y2="20.32" width="0.1524" layer="91"/>
-<pinref part="+3V1" gate="G$1" pin="+3V3"/>
-<wire x1="175.26" y1="20.32" x2="175.26" y2="48.26" width="0.1524" layer="91"/>
-<pinref part="U2" gate="A" pin="!SHDN"/>
-<wire x1="99.06" y1="33.02" x2="99.06" y2="45.72" width="0.1524" layer="91"/>
-<wire x1="99.06" y1="45.72" x2="175.26" y2="45.72" width="0.1524" layer="91"/>
-<wire x1="175.26" y1="45.72" x2="175.26" y2="48.26" width="0.1524" layer="91"/>
-<junction x="175.26" y="48.26"/>
-</segment>
-<segment>
 <pinref part="+3V2" gate="G$1" pin="+3V3"/>
 <pinref part="U3" gate="A" pin="VCC"/>
 <wire x1="160.02" y1="-27.94" x2="154.94" y2="-27.94" width="0.1524" layer="91"/>
+</segment>
+<segment>
+<pinref part="U2" gate="A" pin="VCC"/>
+<pinref part="+3V1" gate="G$1" pin="+3V3"/>
+<wire x1="154.94" y1="27.94" x2="154.94" y2="25.4" width="0.1524" layer="91"/>
+<wire x1="154.94" y1="25.4" x2="160.02" y2="25.4" width="0.1524" layer="91"/>
+</segment>
+<segment>
+<pinref part="U2" gate="A" pin="!SHDN"/>
+<pinref part="C5" gate="G$1" pin="1"/>
+<wire x1="99.06" y1="33.02" x2="99.06" y2="38.1" width="0.1524" layer="91"/>
+<wire x1="99.06" y1="38.1" x2="93.98" y2="38.1" width="0.1524" layer="91"/>
+<pinref part="+3V3" gate="G$1" pin="+3V3"/>
+<wire x1="93.98" y1="38.1" x2="88.9" y2="38.1" width="0.1524" layer="91"/>
+<wire x1="88.9" y1="38.1" x2="88.9" y2="43.18" width="0.1524" layer="91"/>
+<junction x="88.9" y="38.1"/>
+<pinref part="C6" gate="G$1" pin="1"/>
+<junction x="93.98" y="38.1"/>
 </segment>
 </net>
@@
 </segment>
 </net>
-<net name="N$1" class="0">
+<net name="TOGGLE" class="0">
 <segment>
 <pinref part="U2" gate="A" pin="VOUT"/>
-<wire x1="99.06" y1="27.94" x2="91.44" y2="27.94" width="0.1524" layer="91"/>
-</segment>
-</net>
+<wire x1="99.06" y1="27.94" x2="96.52" y2="27.94" width="0.1524" layer="91"/>
+</segment>
+</net>
+<net name="N$2" class="0">
+<segment>
+<pinref part="U2" gate="A" pin="RFIN"/>
+<pinref part="C4" gate="G$1" pin="2"/>
+<wire x1="154.94" y1="35.56" x2="154.94" y2="33.02" width="0.1524" layer="91"/>
+</segment>
+</net>
